File: Hardware/ED Package (Electrical)/KiCad File Drafts/KnifeBotPCB_Draft3/KnifeBotPCB_Draft3_Sensors#2.kicad_sch (KiCad schematic)
At the start: 13 parts, among them J10 Teensy 4.1, J11 DO OEM Board, J13 EZO-EC OEM Board, J14 Leak Sensor #1, J15 Leak Sensor #2, J16 Leak Sensor #3, J17 IMU/InternalPressure, J18 DO Meter, J19 Conductivity Meter, J5 UW Pressure Meter, J7 GPS, J8 Temp Meter

Commit message: End of first day; began poller.py development
Connections:
- net at J7.2 (PPS): now also J10.28 (RX)
