File: Hardware/ED Package (Electrical)/KiCad File Drafts/KnifeBotPCB_Draft3/KnifeBotPCB_Draft3_Unit#2_SCH.kicad_sch (KiCad schematic)
At the start: 48 parts, among them J1 CM5 Raspberry Pi, J12 Raspberry Pi cam module 3, J2 Raspberry_Pi_2_3, J4 TLV7031, J6 XT90PW-M, J9 HaLow Module, Q1 F5305S PMOS, Q2 BSS138 NMOS, SW1 SW_Reed, U1 AP64501SP-13

Commit message: End of first day; began poller.py development
Parts:
- J3: value ~ -> (none)
Connections:
- net ~10mA: now also J1.2 (5V), J1.4 (5V)
